File: eagle/mml_mcu.sch (EAGLE design)
At the start: 52 parts, among them M201 G1040003D, U101 SAMD21E18A-AUT, U201 VEML7700-TT, U202 DRV2605LDGS, U203 LIS2DTW12, U204 74LVC1G125-SOT753, U205 SPX3819SOT-23-5, X101 M50-3600542R, X201 217182-0001, X202 SSM-102-S-DV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

Commit message: MCU board revision B
Parts:
- added PB101: KMR2XXG, xul:KMR2XXG
- C101, C102: value 8p -> 16p
- C207: value 4n7 1kV -> 4n7 250V
- R104: value 470R -> 1k
- TP1, TP2, TP3, TP4, TP5, TP6: value TPTP20R -> TPTP15R; device testpad:TPTP20R -> testpad:TPTP15R
- U205: value SPX3819SOT-23-5 -> MIC5216-3.3YM5-TR
- X202, X203, X204, X205: value SSM-102-S-DV -> HW-02-10-T-D-500-SM; device xul:SSM-102-S-DV -> xul:HW-02-10-T-D-500-SM
- XTAL101: value CM41532768DZCT -> ABS09-32.768KHZ-1-T
- renumbered PB1 to PB102
Connections:
- net /RESET: now also PB101.1
- net GND: now also PB101.2, PB101.5, X202G$2.SK; no longer X202G$4.SK
- net MATRIX_DATA: now also X202G$4.SK; no longer X202G$2.SK
Other:
- note added: "HW-02-12-G-D-710-SM"
- note removed: "Pin layout from Mattairtech MT-D21E https://github.com/mattairtech/ArduinoCore-samd/blob/master/variants/MT_D21E/README.md"
- moved on the sheet: TP1, TP2, TP3, TP4, TP5, TP6
